File: LED Dimmer.kicad_pcb (KiCad board)
At the start: 2 copper layers, 118.1 x 74.9 mm, 78 parts, among them P1 Red Load, P2 Green Load, P3 Blue Load, P4 PWR, Q1 TIP31C, Q2 TIP31C, Q3 TIP31C, Q4 Q_PNP_EBC, Q5 Q_PNP_EBC, Q6 Q_NPN_EBC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

Commit message: Added mounting holes for M3 screws and re-routed accordingly
Parts:
- added REF**: Mounting_Hole, led_dimmer_footprints:Mounting_Hole, F.Cu at (108.7, 136.4)
- added REF**: Mounting_Hole, led_dimmer_footprints:Mounting_Hole, F.Cu at (187.7, 128.0)
- added REF**: Mounting_Hole, led_dimmer_footprints:Mounting_Hole, F.Cu at (186.2, 52.6)
- added REF**: Mounting_Hole, led_dimmer_footprints:Mounting_Hole, F.Cu at (106.7, 51.6)
Routing:
- net GND: track 335.7 -> 340.9 mm
Changed lines of the file:
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@@
     (links 144)
     (no_connects 0)
-    (area 87.579999 46.939999 205.790001 121.970001)
+    (area 87.007699 46.5678 206.362301 121.970001)
     (thickness 1.6)
     (drawings 17)
-    (tracks 517)
+    (tracks 525)
     (zones 0)
-    (modules 78)
+    (modules 82)
     (nets 62)
   )
@@
     (mod_text_size 1 1)
     (mod_text_width 0.15)
-    (pad_size 1.8288 1.8288)
-    (pad_drill 0.762)
+    (pad_size 3.429 3.429)
+    (pad_drill 3.429)
     (pad_to_mask_clearance 0)
     (aux_axis_origin 0 0)
@@
     (add_net "Net-(P3-Pad2)")
   )
+  (module led_dimmer_footprints:Mounting_Hole (layer F.Cu)
+    (at 108.712 136.398)
+    (fp_text reference REF** (at 0 0.5) (layer F.SilkS) hide
+      (effects (font (size 1 1) (thickness 0.15)))
+    )
+    (fp_text value Mounting_Hole (at 0 -0.5) (layer F.Fab) hide
+      (effects (font (size 1 1) (thickness 0.15)))
+    )
+    (pad "" np_thru_hole circle (at -2.032 -19.05) (size 3.429 3.429) (drill 3.429) (layers *.Cu *.Mask))
+  )
+  (module led_dimmer_footprints:Mounting_Hole (layer F.Cu)
+    (at 187.706 128.016)
+    (fp_text reference REF** (at 0 0.5) (layer F.SilkS) hide
+      (effects (font (size 1 1) (thickness 0.15)))
+    )
+    (fp_text value Mounting_Hole (at 0 -0.5) (layer F.Fab) hide
+      (effects (font (size 1 1) (thickness 0.15)))
+    )
+    (pad "" np_thru_hole circle (at -1.524 -10.668) (size 3.429 3.429) (drill 3.429) (layers *.Cu *.Mask))
+  )
+  (module led_dimmer_footprints:Mounting_Hole (layer F.Cu)
+    (at 186.182 52.578)
+    (fp_text reference REF** (at 0 0.5) (layer F.SilkS) hide
+      (effects (font (size 1 1) (thickness 0.15)))
+    )
+    (fp_text value Mounting_Hole (at 0 -0.5) (layer F.Fab) hide
+      (effects (font (size 1 1) (thickness 0.15)))
+    )
+    (pad "" np_thru_hole circle (at 0.508 -1.016) (size 3.429 3.429) (drill 3.429) (layers *.Cu *.Mask))
+  )
   (module led_dimmer_footprints:C_Disc (layer B.Cu)
     (at 94.615 63.5 180)
@@
     )
   )
+  (module led_dimmer_footprints:Mounting_Hole (layer F.Cu)
+    (at 106.68 51.562)
+    (fp_text reference REF** (at 0 0.5) (layer F.SilkS) hide
+      (effects (font (size 1 1) (thickness 0.15)))
+    )
+    (fp_text value Mounting_Hole (at 0 -0.5) (layer F.Fab) hide
+      (effects (font (size 1 1) (thickness 0.15)))
+    )
+    (pad "" np_thru_hole circle (at 0 0) (size 3.429 3.429) (drill 3.429) (layers *.Cu *.Mask))
+  )
   (gr_text RABG (at 101.092 67.564) (layer F.SilkS)
     (effects (font (size 1.5 1.5) (thickness 0.3)))
@@
   (segment (start 148.0006 50.8) (end 139.7456 59.055) (width 0.254) (layer F.Cu) (net 1))
   (segment (start 152.4 50.8) (end 148.0006 50.8) (width 0.254) (layer F.Cu) (net 1))
+  (segment (start 112.395 117.9195) (end 110.9345 117.9195) (width 0.508) (layer F.Cu) (net 2) (status 400000))
+  (segment (start 100.9396 120.142) (end 98.425 117.6274) (width 0.508) (layer F.Cu) (net 2) (status 800000))
+  (segment (start 108.712 120.142) (end 100.9396 120.142) (width 0.508) (layer F.Cu) (net 2))
+  (segment (start 110.9345 117.9195) (end 108.712 120.142) (width 0.508) (layer F.Cu) (net 2))
+  (segment (start 191.008 118.11) (end 187.452 114.554) (width 0.508) (layer F.Cu) (net 2))
+  (segment (start 194.564 118.11) (end 191.008 118.11) (width 0.508) (layer F.Cu) (net 2))
+  (segment (start 139.7 118.11) (end 181.102 118.11) (width 0.508) (layer F.Cu) (net 2))
+  (segment (start 187.452 114.554) (end 184.658 114.554) (width 0.508) (layer F.Cu) (net 2))
+  (segment (start 184.658 114.554) (end 181.102 118.11) (width 0.508) (layer F.Cu) (net 2))
   (segment (start 115.1685 55.0115) (end 115.57 54.61) (width 0.508) (layer B.Cu) (net 2))
   (segment (start 113.665 56.515) (end 115.1685 55.0115) (width 0.508) (layer B.Cu) (net 2))
@@
   (segment (start 137.7885 118.11) (end 136.2547 119.6438) (width 0.508) (layer F.Cu) (net 2))
   (segment (start 98.7171 117.9195) (end 98.425 117.6274) (width 0.508) (layer F.Cu) (net 2))
-  (segment (start 112.395 117.9195) (end 98.7171 117.9195) (width 0.508) (layer F.Cu) (net 2))
   (segment (start 92.075 58.8645) (end 92.075 63.5) (width 0.508) (layer B.Cu) (net 2))
   (segment (start 91.44 58.2295) (end 92.075 58.8645) (width 0.508) (layer B.Cu) (net 2))
   (segment (start 194.6035 118.11) (end 194.564 118.11) (width 0.508) (layer F.Cu) (net 2))
-  (segment (start 194.564 118.11) (end 139.7 118.11) (width 0.508) (layer F.Cu) (net 2))
   (segment (start 103.892 70.8785) (end 105.4035 72.39) (width 0.508) (layer F.Cu) (net 2))
   (segment (start 92.699 70.8785) (end 103.892 70.8785) (width 0.508) (layer F.Cu) (net 2))
@@
   (segment (start 195.7742 111.125) (end 188.0725 103.4233) (width 0.254) (layer F.Cu) (net 14))
   (segment (start 198.12 111.125) (end 195.7742 111.125) (width 0.254) (layer F.Cu) (net 14))
+  (segment (start 104.775 54.8005) (end 106.9975 54.8005) (width 0.254) (layer F.Cu) (net 15))
+  (segment (start 106.9975 54.8005) (end 108.5092 53.2888) (width 0.254) (layer F.Cu) (net 15))
   (segment (start 100.33 54.8005) (end 104.775 54.8005) (width 0.254) (layer F.Cu) (net 15))
   (segment (start 129.4888 53.2888) (end 132.715 56.515) (width 0.254) (layer F.Cu) (net 15))
-  (segment (start 106.2867 53.2888) (end 129.4888 53.2888) (width 0.254) (layer F.Cu) (net 15))
-  (segment (start 104.775 54.8005) (end 106.2867 53.2888) (width 0.254) (layer F.Cu) (net 15))
+  (segment (start 108.5092 53.2888) (end 129.4888 53.2888) (width 0.254) (layer F.Cu) (net 15))
   (segment (start 125.5332 56.515) (end 128.27 56.515) (width 0.254) (layer B.Cu) (net 16))
   (segment (start 122.9932 59.055) (end 125.5332 56.515) (width 0.254) (layer B.Cu) (net 16))

Commit message: Copper pour, maybe
Routing:
- added copper zone on B.Cu, net GND
- added copper zone on F.Cu, net GND
Changed lines of the file:
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@@
     (links 144)
     (no_connects 0)
-    (area 87.007699 46.5678 206.362301 121.970001)
+    (area 87.007699 46.5678 206.362301 138.2302)
     (thickness 1.6)
     (drawings 17)
@@
     (visible_elements 7FFFFFFF)
     (pcbplotparams
-      (layerselection 0x00030_80000001)
+      (layerselection 0x010f0_80000001)
       (usegerberextensions false)
       (excludeedgelayer true)
@@
       (outputformat 1)
       (mirror false)
-      (drillshape 1)
+      (drillshape 0)
       (scaleselection 1)
-      (outputdirectory ""))
+      (outputdirectory Gerbs/))
   )
   (net 0 "")
@@
   (segment (start 101.4795 101.7205) (end 100.965 102.235) (width 0.254) (layer B.Cu) (net 47))
   (segment (start 101.4795 78.8735) (end 101.4795 101.7205) (width 0.254) (layer B.Cu) (net 47))
+  (zone (net 2) (net_name GND) (layer F.Cu) (hatch edge 0.508)
+    (connect_pads (clearance 0.508))
+    (min_thickness 0.254)
+    (fill (arc_segments 16) (thermal_gap 0.508) (thermal_bridge_width 0.508))
+    (polygon
+      (pts
+        (xy 205.74 121.92) (xy 87.63 121.92) (xy 87.63 46.99) (xy 205.74 46.99)
+      )
+    )
+  )
+  (zone (net 2) (net_name GND) (layer B.Cu) (hatch edge 0.508)
+    (connect_pads (clearance 0.508))
+    (min_thickness 0.254)
+    (fill (arc_segments 16) (thermal_gap 0.508) (thermal_bridge_width 0.508))
+    (polygon
+      (pts
+        (xy 205.74 121.92) (xy 87.63 121.92) (xy 87.63 46.99) (xy 205.74 46.99)
+      )
+    )
+  )
 )
