File: LED Dimmer.kicad_pcb (KiCad board)
At the start: 2 copper layers, 118.1 x 74.9 mm, 82 parts, among them P1 Red Load, P2 Green Load, P3 Blue Load, P4 PWR, Q1 TIP31C, Q2 TIP31C, Q3 TIP31C, Q4 Q_PNP_EBC, Q5 Q_PNP_EBC, Q6 Q_NPN_EBC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

Commit message: Finished front panel, I think
Other:
- board text added: "samsam loves penny!!!!!!"
Changed lines of the file:
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@@
     (links 144)
     (no_connects 0)
-    (area 87.007699 46.5678 206.362301 138.2302)
+    (area 69.949287 42.672 212.852001 138.2302)
     (thickness 1.6)
-    (drawings 16)
+    (drawings 19)
     (tracks 525)
     (zones 0)
@@
     (47 F.CrtYd user hide)
     (48 B.Fab user hide)
-    (49 F.Fab user hide)
+    (49 F.Fab user)
   )
   (setup
@@
     (pad "" np_thru_hole circle (at 0 0) (size 3.2004 3.2004) (drill 3.2004) (layers *.Cu *.Mask))
   )
+  (gr_text "samsam loves penny!!!!!!" (at 165.1 95.25) (layer F.SilkS)
+    (effects (font (size 1.5 1.5) (thickness 0.3)))
+  )
+  (dimension 74.93 (width 0.3) (layer F.Fab)
+    (gr_text "2.9500 in" (at 75.485 84.455 90) (layer F.Fab)
+      (effects (font (size 1.5 1.5) (thickness 0.3)))
+    )
+    (feature1 (pts (xy 87.63 46.99) (xy 74.135 46.99)))
+    (feature2 (pts (xy 87.63 121.92) (xy 74.135 121.92)))
+    (crossbar (pts (xy 76.835 121.92) (xy 76.835 46.99)))
+    (arrow1a (pts (xy 76.835 46.99) (xy 77.421421 48.116504)))
+    (arrow1b (pts (xy 76.835 46.99) (xy 76.248579 48.116504)))
+    (arrow2a (pts (xy 76.835 121.92) (xy 77.421421 120.793496)))
+    (arrow2b (pts (xy 76.835 121.92) (xy 76.248579 120.793496)))
+  )
+  (dimension 118.11 (width 0.3) (layer F.Fab)
+    (gr_text "4.6500 in" (at 146.685 129.62) (layer F.Fab)
+      (effects (font (size 1.5 1.5) (thickness 0.3)))
+    )
+    (feature1 (pts (xy 87.63 121.92) (xy 87.63 130.97)))
+    (feature2 (pts (xy 205.74 121.92) (xy 205.74 130.97)))
+    (crossbar (pts (xy 205.74 128.27) (xy 87.63 128.27)))
+    (arrow1a (pts (xy 87.63 128.27) (xy 88.756504 127.683579)))
+    (arrow1b (pts (xy 87.63 128.27) (xy 88.756504 128.856421)))
+    (arrow2a (pts (xy 205.74 128.27) (xy 204.613496 127.683579)))
+    (arrow2b (pts (xy 205.74 128.27) (xy 204.613496 128.856421)))
+  )
   (gr_arc (start 90.17 119.38) (end 90.17 121.92) (angle 90) (layer Edge.Cuts) (width 0.1))
