File: front panel.kicad_pcb (KiCad board)
At the start: 2 copper layers, 118.1 x 74.9 mm, 18 parts, among them SW1 SW_SPDT, SW10 SW_SPDT, SW11 SW_SPDT, SW12 SW_SPDT, SW2 SW_SPDT, SW3 SW_SPDT, SW4 SW_SPDT, SW5 SW_SPDT, SW6 SW_SPDT, SW7 SW_SPDT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

Commit message: Finished front panel, I think
Parts:
- added G***: LOGO, led_dimmer_footprints:smallbab, F.Cu at (120.0, 71.8)
- added G***: LOGO, led_dimmer_footprints:irish2, F.Cu at (146.7, 84.1)
